File: pcb/KOMETA.kicad_pcb (KiCad board)
At the start: 2 copper layers, 279.2 x 87.1 mm, 119 parts

Commit message: update silkscreen
Other:
- board text added: "designed by: inpudiy customkey turtle torowb"
- board text removed: "designed by: inpudiy customkey turtle"

Commit message: update silkscreen
Parts:
- removed ? (x4): , 
- added G***: LOGO, LOGO, B.Cu at (70.5, 151.0)
- added G***: LOGO, LOGO, B.Cu at (298.9, 131.5)
- added G***: LOGO, LOGO, B.Cu at (135.3, 126.8)
- added G***: LOGO, LOGO, B.Cu at (279.9, 126.8)
- added G***: LOGO, LOGO, B.Cu at (344.1, 170.0)
- added G***: LOGO, LOGO, B.Cu at (241.9, 133.9)
- added G***: LOGO, LOGO, B.Cu at (70.5, 132.0)
- added G***: LOGO, LOGO, B.Cu at (344.1, 151.0)
- added G***: LOGO, LOGO, B.Cu at (268.1, 179.5)
- added G***: LOGO, LOGO, B.Cu at (116.3, 131.5)
- added G***: LOGO, LOGO, B.Cu at (70.5, 170.0)
- added G***: LOGO, LOGO, B.Cu at (97.3, 138.7)
- added G***: LOGO, LOGO, B.Cu at (146.5, 179.5)
- added G***: LOGO, LOGO, B.Cu at (260.9, 131.5)
- added G***: LOGO, LOGO, B.Cu at (317.9, 138.7)
- added G***: LOGO, LOGO, B.Cu at (173.3, 133.9)
- added G***: LOGO, LOGO, B.Cu at (154.3, 131.5)
- added G***: LOGO, LOGO, B.Cu at (344.1, 132.0)
- added G***: LOGO, LOGO, B.Cu at (78.3, 141.0)
- added G***: LOGO, LOGO, B.Cu at (336.9, 140.0)
Other:
- board text added: "C0"
- board text added: "C1"
- board text added: "C2"
- board text added: "C3"
- board text added: "C4"
- board text added: "C5"
- board text added: "Case: toworb & customkey"
- board text added: "KOMETA"
- board text added: "LEFT DOWN"
- board text added: "LEFT UP"
- board text added: "PCB: inpudiy & turtle"
- board text added: "R0"
- board text added: "R1"
- board text added: "R2"
- board text added: "R3"
- board text added: "RIGHT DOWN"
- board text added: "RIGHT UP"
- board text added: "V0.9.9"
- board text removed: "c0"
- board text removed: "c1"
- board text removed: "c2"
- board text removed: "c3"
- board text removed: "c4"
- board text removed: "c5"
- board text removed: "designed by: inpudiy customkey turtle torowb"
- board text removed: "left down"
- board text removed: "left up"
- board text removed: "r0"
- board text removed: "r1"
- board text removed: "r2"
- board text removed: "r3"
- board text removed: "right down"
- board text removed: "right up"
