File: pcb/KOMETA.kicad_sch (KiCad schematic)
At the start: 13 parts

Commit message: add support choc v1
Parts:
- H1, H10, H11, H12, H2, H3, H4, H5, H6, H7, H8, H9: footprint lib:M2 Hole -> kometa:M2 Hole
- KeyChainHole1: footprint lib:M5 hole -> kometa:M5 hole
Changed lines of the file:
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@@
 			)
 		)
-		(property "Footprint" "lib:M2 Hole"
+		(property "Footprint" "kometa:M2 Hole"
 			(at 16.51 177.8 0)
 			(effects
@@
 			)
 		)
-		(property "Footprint" "lib:M2 Hole"
+		(property "Footprint" "kometa:M2 Hole"
 			(at 26.67 187.96 0)
 			(effects
@@
 			)
 		)
-		(property "Footprint" "lib:M2 Hole"
+		(property "Footprint" "kometa:M2 Hole"
 			(at 26.67 177.8 0)
 			(effects
@@
 			)
 		)
-		(property "Footprint" "lib:M2 Hole"
+		(property "Footprint" "kometa:M2 Hole"
 			(at 26.67 193.04 0)
 			(effects
@@
 			)
 		)
-		(property "Footprint" "lib:M5 hole"
+		(property "Footprint" "kometa:M5 hole"
 			(at 16.51 162.56 0)
 			(effects
@@
 			)
 		)
-		(property "Footprint" "lib:M2 Hole"
+		(property "Footprint" "kometa:M2 Hole"
 			(at 26.67 172.72 0)
 			(effects
@@
 			)
 		)
-		(property "Footprint" "lib:M2 Hole"
+		(property "Footprint" "kometa:M2 Hole"
 			(at 26.67 182.88 0)
 			(effects
@@
 			)
 		)
-		(property "Footprint" "lib:M2 Hole"
+		(property "Footprint" "kometa:M2 Hole"
 			(at 26.67 167.64 0)
 			(effects
@@
 			)
 		)
-		(property "Footprint" "lib:M2 Hole"
+		(property "Footprint" "kometa:M2 Hole"
 			(at 16.51 172.72 0)
 			(effects
@@
 			)
 		)
-		(property "Footprint" "lib:M2 Hole"
+		(property "Footprint" "kometa:M2 Hole"
 			(at 16.51 167.64 0)
 			(effects
@@
 			)
 		)
-		(property "Footprint" "lib:M2 Hole"
+		(property "Footprint" "kometa:M2 Hole"
 			(at 16.51 193.04 0)
 			(effects
@@
 			)
 		)
-		(property "Footprint" "lib:M2 Hole"
+		(property "Footprint" "kometa:M2 Hole"
 			(at 16.51 182.88 0)
 			(effects
@@
 			)
 		)
-		(property "Footprint" "lib:M2 Hole"
+		(property "Footprint" "kometa:M2 Hole"
 			(at 16.51 187.96 0)
 			(effects

Commit message: update footprint
Parts:
- H1, H10, H11, H12, H2, H3, H4, H5, H6, H7, H8, H9: footprint kometa:M2 Hole -> lib:M2 Hole
- KeyChainHole1: footprint kometa:M5 hole -> lib:M5 hole
Changed lines of the file:
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@@
 			)
 		)
-		(property "Footprint" "kometa:M2 Hole"
+		(property "Footprint" "lib:M2 Hole"
 			(at 16.51 177.8 0)
 			(effects
@@
 			)
 		)
-		(property "Footprint" "kometa:M2 Hole"
+		(property "Footprint" "lib:M2 Hole"
 			(at 26.67 187.96 0)
 			(effects
@@
 			)
 		)
-		(property "Footprint" "kometa:M2 Hole"
+		(property "Footprint" "lib:M2 Hole"
 			(at 26.67 177.8 0)
 			(effects
@@
 			)
 		)
-		(property "Footprint" "kometa:M2 Hole"
+		(property "Footprint" "lib:M2 Hole"
 			(at 26.67 193.04 0)
 			(effects
@@
 			)
 		)
-		(property "Footprint" "kometa:M5 hole"
+		(property "Footprint" "lib:M5 hole"
 			(at 16.51 162.56 0)
 			(effects
@@
 			)
 		)
-		(property "Footprint" "kometa:M2 Hole"
+		(property "Footprint" "lib:M2 Hole"
 			(at 26.67 172.72 0)
 			(effects
@@
 			)
 		)
-		(property "Footprint" "kometa:M2 Hole"
+		(property "Footprint" "lib:M2 Hole"
 			(at 26.67 182.88 0)
 			(effects
@@
 			)
 		)
-		(property "Footprint" "kometa:M2 Hole"
+		(property "Footprint" "lib:M2 Hole"
 			(at 26.67 167.64 0)
 			(effects
@@
 			)
 		)
-		(property "Footprint" "kometa:M2 Hole"
+		(property "Footprint" "lib:M2 Hole"
 			(at 16.51 172.72 0)
 			(effects
@@
 			)
 		)
-		(property "Footprint" "kometa:M2 Hole"
+		(property "Footprint" "lib:M2 Hole"
 			(at 16.51 167.64 0)
 			(effects
@@
 			)
 		)
-		(property "Footprint" "kometa:M2 Hole"
+		(property "Footprint" "lib:M2 Hole"
 			(at 16.51 193.04 0)
 			(effects
@@
 			)
 		)
-		(property "Footprint" "kometa:M2 Hole"
+		(property "Footprint" "lib:M2 Hole"
 			(at 16.51 182.88 0)
 			(effects
@@
 			)
 		)
-		(property "Footprint" "kometa:M2 Hole"
+		(property "Footprint" "lib:M2 Hole"
 			(at 16.51 187.96 0)
 			(effects
