File: pcb/left.kicad_sch (KiCad schematic)
At the start: 46 parts

Commit message: add support choc v1
Parts:
- D1, D10, D11, D12, D13, D14, D15, D16, D17, D18, D19, D2, D20, D21, D3, D4, D5, D6, D7, D8, D9: footprint lib:Diode -> kometa:Diode
- PS_L1: footprint lib:MSK-12C02 -> kometa:MSK-12C02
- PW_L1: footprint lib:Battery -> kometa:Battery
- R_L1: footprint lib:Reset -> kometa:Reset
- SM_L1: footprint lib:SuperMini -> kometa:SuperMini
- SW1, SW10, SW11, SW12, SW13, SW14, SW15, SW16, SW17, SW18, SW19, SW2, SW20, SW21, SW3, SW4, SW5, SW6, SW7, SW8, SW9: footprint lib:ChocV2 -> kometa:ChocV2
Changed lines of the file:
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@@
 			)
 		)
-		(property "Footprint" "lib:ChocV2"
+		(property "Footprint" "kometa:ChocV2"
 			(at 79.756 105.41 0)
 			(effects
@@
 			)
 		)
-		(property "Footprint" "lib:ChocV2"
+		(property "Footprint" "kometa:ChocV2"
 			(at 136.906 105.41 0)
 			(effects
@@
 			)
 		)
-		(property "Footprint" "lib:ChocV2"
+		(property "Footprint" "kometa:ChocV2"
 			(at 41.656 86.36 0)
 			(effects
@@
 			)
 		)
-		(property "Footprint" "lib:Diode"
+		(property "Footprint" "kometa:Diode"
 			(at 138.176 102.362 0)
 			(effects
@@
 			)
 		)
-		(property "Footprint" "lib:ChocV2"
+		(property "Footprint" "kometa:ChocV2"
 			(at 136.906 86.36 0)
 			(effects
@@
 			)
 		)
-		(property "Footprint" "lib:Diode"
+		(property "Footprint" "kometa:Diode"
 			(at 61.976 83.312 0)
 			(effects
@@
 			)
 		)
-		(property "Footprint" "lib:Battery"
+		(property "Footprint" "kometa:Battery"
 			(at 176.784 78.486 0)
 			(effects
@@
 			)
 		)
-		(property "Footprint" "lib:Diode"
+		(property "Footprint" "kometa:Diode"
 			(at 81.026 102.362 0)
 			(effects
@@
 			)
 		)
-		(property "Footprint" "lib:ChocV2"
+		(property "Footprint" "kometa:ChocV2"
 			(at 98.806 124.46 0)
 			(effects
@@
 			)
 		)
-		(property "Footprint" "lib:ChocV2"
+		(property "Footprint" "kometa:ChocV2"
 			(at 136.906 124.46 0)
 			(effects
@@
 			)
 		)
-		(property "Footprint" "lib:ChocV2"
+		(property "Footprint" "kometa:ChocV2"
 			(at 60.706 86.36 0)
 			(effects
@@
 			)
 		)
-		(property "Footprint" "lib:ChocV2"
+		(property "Footprint" "kometa:ChocV2"
 			(at 117.856 144.78 0)
 			(effects
@@
 			)
 		)
-		(property "Footprint" "lib:Diode"
+		(property "Footprint" "kometa:Diode"
 			(at 100.076 141.732 0)
 			(effects
@@
 			)
 		)
-		(property "Footprint" "lib:ChocV2"
+		(property "Footprint" "kometa:ChocV2"
 			(at 117.856 105.41 0)
 			(effects
@@
 			)
 		)
-		(property "Footprint" "lib:ChocV2"
+		(property "Footprint" "kometa:ChocV2"
 			(at 79.756 86.36 0)
 			(effects
@@
 			)
 		)
-		(property "Footprint" "lib:Diode"
+		(property "Footprint" "kometa:Diode"
 			(at 119.126 141.732 0)
 			(effects
@@
 			)
 		)
-		(property "Footprint" "lib:Diode"
+		(property "Footprint" "kometa:Diode"
 			(at 81.026 121.412 0)
 			(effects
@@
 			)
 		)
-		(property "Footprint" "lib:Reset"
+		(property "Footprint" "kometa:Reset"
 			(at 185.42 102.87 0)
 			(effects
@@
 			)
 		)
-		(property "Footprint" "lib:Diode"
+		(property "Footprint" "kometa:Diode"
 			(at 81.026 83.312 0)
 			(effects
@@
 			)
 		)
-		(property "Footprint" "lib:Diode"
+		(property "Footprint" "kometa:Diode"
 			(at 119.126 102.362 0)
 			(effects
@@
 			)
 		)
-		(property "Footprint" "lib:Diode"
+		(property "Footprint" "kometa:Diode"
 			(at 138.176 121.412 0)
 			(effects
@@
 			)
 		)
-		(property "Footprint" "lib:Diode"
+		(property "Footprint" "kometa:Diode"
 			(at 42.926 83.312 0)
 			(effects
@@
 			)
 		)
-		(property "Footprint" "lib:Diode"
+		(property "Footprint" "kometa:Diode"
 			(at 42.926 121.412 0)
 			(effects
@@
 			)
 		)
-		(property "Footprint" "lib:ChocV2"
+		(property "Footprint" "kometa:ChocV2"
 			(at 117.856 86.36 0)
 			(effects
@@
 			)
 		)
-		(property "Footprint" "lib:Diode"
+		(property "Footprint" "kometa:Diode"
 			(at 119.126 121.412 0)
 			(effects
@@
 			)
 		)
-		(property "Footprint" "lib:ChocV2"
+		(property "Footprint" "kometa:ChocV2"
 			(at 41.656 124.46 0)
 			(effects
@@
 			)
 		)
-		(property "Footprint" "lib:Diode"
+		(property "Footprint" "kometa:Diode"
 			(at 138.176 83.312 0)
 			(effects
@@
 			)
 		)
-		(property "Footprint" "lib:ChocV2"
+		(property "Footprint" "kometa:ChocV2"
 			(at 60.706 124.46 0)
 			(effects
@@
 			)
 		)
-		(property "Footprint" "lib:Diode"
+		(property "Footprint" "kometa:Diode"
 			(at 61.976 102.362 0)
 			(effects
@@
 			)
 		)
-		(property "Footprint" "lib:ChocV2"
+		(property "Footprint" "kometa:ChocV2"
 			(at 98.806 86.36 0)
 			(effects
@@
 			)
 		)
-		(property "Footprint" "lib:ChocV2"
+		(property "Footprint" "kometa:ChocV2"
 			(at 117.856 124.46 0)
 			(effects
@@
 			)
 		)
-		(property "Footprint" "lib:ChocV2"
+		(property "Footprint" "kometa:ChocV2"
 			(at 98.806 144.78 0)
 			(effects
@@
 			)
 		)
-		(property "Footprint" "lib:ChocV2"
+		(property "Footprint" "kometa:ChocV2"
 			(at 41.656 105.41 0)
 			(effects
@@
 			)
 		)
-		(property "Footprint" "lib:Diode"
+		(property "Footprint" "kometa:Diode"
 			(at 138.176 141.732 0)
 			(effects
@@
 			)
 		)
-		(property "Footprint" "lib:Diode"
+		(property "Footprint" "kometa:Diode"
 			(at 119.126 83.312 0)
 			(effects
@@
 			)
 		)
-		(property "Footprint" "lib:ChocV2"
+		(property "Footprint" "kometa:ChocV2"
 			(at 60.706 105.41 0)
 			(effects
@@
 			)
 		)
-		(property "Footprint" "lib:ChocV2"
+		(property "Footprint" "kometa:ChocV2"
 			(at 98.806 105.41 0)
 			(effects
@@
 			)
 		)
-		(property "Footprint" "lib:ChocV2"
+		(property "Footprint" "kometa:ChocV2"
 			(at 79.756 124.46 0)
 			(effects
@@
 			)
 		)
-		(property "Footprint" "lib:SuperMini"
+		(property "Footprint" "kometa:SuperMini"
 			(at 241.3 109.728 0)
 			(effects
@@
 			)
 		)
-		(property "Footprint" "lib:Diode"
+		(property "Footprint" "kometa:Diode"
 			(at 61.976 121.412 0)
 			(effects
@@
 			)
 		)
-		(property "Footprint" "lib:MSK-12C02"
+		(property "Footprint" "kometa:MSK-12C02"
 			(at 186.944 80.264 0)
 			(effects
@@
 			)
 		)
-		(property "Footprint" "lib:Diode"
+		(property "Footprint" "kometa:Diode"
 			(at 100.076 83.312 0)
 			(effects
@@
 			)
 		)
-		(property "Footprint" "lib:ChocV2"
+		(property "Footprint" "kometa:ChocV2"
 			(at 136.906 144.78 0)
 			(effects
@@
 			)
 		)
-		(property "Footprint" "lib:Diode"
+		(property "Footprint" "kometa:Diode"
 			(at 100.076 121.412 0)
 			(effects
@@
 			)
 		)
-		(property "Footprint" "lib:Diode"
+		(property "Footprint" "kometa:Diode"
 			(at 42.926 102.362 0)
 			(effects
@@
 			)
 		)
-		(property "Footprint" "lib:Diode"
+		(property "Footprint" "kometa:Diode"
 			(at 100.076 102.362 0)
 			(effects

Commit message: update footprint
Parts:
- D1, D10, D11, D12, D13, D14, D15, D16, D17, D18, D19, D2, D20, D21, D3, D4, D5, D6, D7, D8, D9: footprint kometa:Diode -> lib:Diode
- PS_L1: footprint kometa:MSK-12C02 -> lib:MSK-12C02
- PW_L1: footprint kometa:Battery -> lib:Battery
- R_L1: footprint kometa:Reset -> lib:Reset
- SM_L1: footprint kometa:SuperMini -> lib:SuperMini
- SW1, SW10, SW11, SW12, SW13, SW14, SW15, SW16, SW17, SW18, SW19, SW2, SW20, SW21, SW3, SW4, SW5, SW6, SW7, SW8, SW9: footprint kometa:ChocV2 -> lib:ChocV2
Changed lines of the file:
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@@
 			)
 		)
-		(property "Footprint" "kometa:ChocV2"
+		(property "Footprint" "lib:ChocV2"
 			(at 79.756 105.41 0)
 			(effects
@@
 			)
 		)
-		(property "Footprint" "kometa:ChocV2"
+		(property "Footprint" "lib:ChocV2"
 			(at 136.906 105.41 0)
 			(effects
@@
 			)
 		)
-		(property "Footprint" "kometa:ChocV2"
+		(property "Footprint" "lib:ChocV2"
 			(at 41.656 86.36 0)
 			(effects
@@
 			)
 		)
-		(property "Footprint" "kometa:Diode"
+		(property "Footprint" "lib:Diode"
 			(at 138.176 102.362 0)
 			(effects
@@
 			)
 		)
-		(property "Footprint" "kometa:ChocV2"
+		(property "Footprint" "lib:ChocV2"
 			(at 136.906 86.36 0)
 			(effects
@@
 			)
 		)
-		(property "Footprint" "kometa:Diode"
+		(property "Footprint" "lib:Diode"
 			(at 61.976 83.312 0)
 			(effects
@@
 			)
 		)
-		(property "Footprint" "kometa:Battery"
+		(property "Footprint" "lib:Battery"
 			(at 176.784 78.486 0)
 			(effects
@@
 			)
 		)
-		(property "Footprint" "kometa:Diode"
+		(property "Footprint" "lib:Diode"
 			(at 81.026 102.362 0)
 			(effects
@@
 			)
 		)
-		(property "Footprint" "kometa:ChocV2"
+		(property "Footprint" "lib:ChocV2"
 			(at 98.806 124.46 0)
 			(effects
@@
 			)
 		)
-		(property "Footprint" "kometa:ChocV2"
+		(property "Footprint" "lib:ChocV2"
 			(at 136.906 124.46 0)
 			(effects
@@
 			)
 		)
-		(property "Footprint" "kometa:ChocV2"
+		(property "Footprint" "lib:ChocV2"
 			(at 60.706 86.36 0)
 			(effects
@@
 			)
 		)
-		(property "Footprint" "kometa:ChocV2"
+		(property "Footprint" "lib:ChocV2"
 			(at 117.856 144.78 0)
 			(effects
@@
 			)
 		)
-		(property "Footprint" "kometa:Diode"
+		(property "Footprint" "lib:Diode"
 			(at 100.076 141.732 0)
 			(effects
@@
 			)
 		)
-		(property "Footprint" "kometa:ChocV2"
+		(property "Footprint" "lib:ChocV2"
 			(at 117.856 105.41 0)
 			(effects
@@
 			)
 		)
-		(property "Footprint" "kometa:ChocV2"
+		(property "Footprint" "lib:ChocV2"
 			(at 79.756 86.36 0)
 			(effects
@@
 			)
 		)
-		(property "Footprint" "kometa:Diode"
+		(property "Footprint" "lib:Diode"
 			(at 119.126 141.732 0)
 			(effects
@@
 			)
 		)
-		(property "Footprint" "kometa:Diode"
+		(property "Footprint" "lib:Diode"
 			(at 81.026 121.412 0)
 			(effects
@@
 			)
 		)
-		(property "Footprint" "kometa:Reset"
+		(property "Footprint" "lib:Reset"
 			(at 185.42 102.87 0)
 			(effects
@@
 			)
 		)
-		(property "Footprint" "kometa:Diode"
+		(property "Footprint" "lib:Diode"
 			(at 81.026 83.312 0)
 			(effects
@@
 			)
 		)
-		(property "Footprint" "kometa:Diode"
+		(property "Footprint" "lib:Diode"
 			(at 119.126 102.362 0)
 			(effects
@@
 			)
 		)
-		(property "Footprint" "kometa:Diode"
+		(property "Footprint" "lib:Diode"
 			(at 138.176 121.412 0)
 			(effects
@@
 			)
 		)
-		(property "Footprint" "kometa:Diode"
+		(property "Footprint" "lib:Diode"
 			(at 42.926 83.312 0)
 			(effects
@@
 			)
 		)
-		(property "Footprint" "kometa:Diode"
+		(property "Footprint" "lib:Diode"
 			(at 42.926 121.412 0)
 			(effects
@@
 			)
 		)
-		(property "Footprint" "kometa:ChocV2"
+		(property "Footprint" "lib:ChocV2"
 			(at 117.856 86.36 0)
 			(effects
@@
 			)
 		)
-		(property "Footprint" "kometa:Diode"
+		(property "Footprint" "lib:Diode"
 			(at 119.126 121.412 0)
 			(effects
@@
 			)
 		)
-		(property "Footprint" "kometa:ChocV2"
+		(property "Footprint" "lib:ChocV2"
 			(at 41.656 124.46 0)
 			(effects
@@
 			)
 		)
-		(property "Footprint" "kometa:Diode"
+		(property "Footprint" "lib:Diode"
 			(at 138.176 83.312 0)
 			(effects
@@
 			)
 		)
-		(property "Footprint" "kometa:ChocV2"
+		(property "Footprint" "lib:ChocV2"
 			(at 60.706 124.46 0)
 			(effects
@@
 			)
 		)
-		(property "Footprint" "kometa:Diode"
+		(property "Footprint" "lib:Diode"
 			(at 61.976 102.362 0)
 			(effects
@@
 			)
 		)
-		(property "Footprint" "kometa:ChocV2"
+		(property "Footprint" "lib:ChocV2"
 			(at 98.806 86.36 0)
 			(effects
@@
 			)
 		)
-		(property "Footprint" "kometa:ChocV2"
+		(property "Footprint" "lib:ChocV2"
 			(at 117.856 124.46 0)
 			(effects
@@
 			)
 		)
-		(property "Footprint" "kometa:ChocV2"
+		(property "Footprint" "lib:ChocV2"
 			(at 98.806 144.78 0)
 			(effects
@@
 			)
 		)
-		(property "Footprint" "kometa:ChocV2"
+		(property "Footprint" "lib:ChocV2"
 			(at 41.656 105.41 0)
 			(effects
@@
 			)
 		)
-		(property "Footprint" "kometa:Diode"
+		(property "Footprint" "lib:Diode"
 			(at 138.176 141.732 0)
 			(effects
@@
 			)
 		)
-		(property "Footprint" "kometa:Diode"
+		(property "Footprint" "lib:Diode"
 			(at 119.126 83.312 0)
 			(effects
@@
 			)
 		)
-		(property "Footprint" "kometa:ChocV2"
+		(property "Footprint" "lib:ChocV2"
 			(at 60.706 105.41 0)
 			(effects
@@
 			)
 		)
-		(property "Footprint" "kometa:ChocV2"
+		(property "Footprint" "lib:ChocV2"
 			(at 98.806 105.41 0)
 			(effects
@@
 			)
 		)
-		(property "Footprint" "kometa:ChocV2"
+		(property "Footprint" "lib:ChocV2"
 			(at 79.756 124.46 0)
 			(effects
@@
 			)
 		)
-		(property "Footprint" "kometa:SuperMini"
+		(property "Footprint" "lib:SuperMini"
 			(at 241.3 109.728 0)
 			(effects
@@
 			)
 		)
-		(property "Footprint" "kometa:Diode"
+		(property "Footprint" "lib:Diode"
 			(at 61.976 121.412 0)
 			(effects
@@
 			)
 		)
-		(property "Footprint" "kometa:MSK-12C02"
+		(property "Footprint" "lib:MSK-12C02"
 			(at 186.944 80.264 0)
 			(effects
@@
 			)
 		)
-		(property "Footprint" "kometa:Diode"
+		(property "Footprint" "lib:Diode"
 			(at 100.076 83.312 0)
 			(effects
@@
 			)
 		)
-		(property "Footprint" "kometa:ChocV2"
+		(property "Footprint" "lib:ChocV2"
 			(at 136.906 144.78 0)
 			(effects
@@
 			)
 		)
-		(property "Footprint" "kometa:Diode"
+		(property "Footprint" "lib:Diode"
 			(at 100.076 121.412 0)
 			(effects
@@
 			)
 		)
-		(property "Footprint" "kometa:Diode"
+		(property "Footprint" "lib:Diode"
 			(at 42.926 102.362 0)
 			(effects
@@
 			)
 		)
-		(property "Footprint" "kometa:Diode"
+		(property "Footprint" "lib:Diode"
 			(at 100.076 102.362 0)
 			(effects
