File: pcb/right.kicad_sch (KiCad schematic)
At the start: 46 parts

Commit message: update footprint
Parts:
- D22, D23, D24, D25, D26, D27, D28, D29, D30, D31, D32, D33, D34, D35, D36, D37, D38, D39, D40, D41, D42: footprint kometa:Diode -> lib:Diode
- PS_R1: footprint kometa:MSK-12C02 -> lib:MSK-12C02
- PW_R1: footprint kometa:Battery -> lib:Battery
- R_R1: footprint kometa:Reset -> lib:Reset
- SM_R1: footprint kometa:SuperMini -> lib:SuperMini
- SW22, SW23, SW24, SW25, SW26, SW27, SW28, SW29, SW30, SW31, SW32, SW33, SW34, SW35, SW36, SW37, SW38, SW39, SW40, SW41, SW42: footprint kometa:ChocV2 -> lib:ChocV2
Changed lines of the file:
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@@
 			)
 		)
-		(property "Footprint" "kometa:ChocV2"
+		(property "Footprint" "lib:ChocV2"
 			(at 64.516 93.98 0)
 			(effects
@@
 			)
 		)
-		(property "Footprint" "kometa:ChocV2"
+		(property "Footprint" "lib:ChocV2"
 			(at 135.636 130.81 0)
 			(effects
@@
 			)
 		)
-		(property "Footprint" "kometa:Diode"
+		(property "Footprint" "lib:Diode"
 			(at 136.906 108.712 0)
 			(effects
@@
 			)
 		)
-		(property "Footprint" "kometa:Diode"
+		(property "Footprint" "lib:Diode"
 			(at 83.566 127.762 0)
 			(effects
@@
 			)
 		)
-		(property "Footprint" "kometa:ChocV2"
+		(property "Footprint" "lib:ChocV2"
 			(at 64.516 111.76 0)
 			(effects
@@
 			)
 		)
-		(property "Footprint" "kometa:Diode"
+		(property "Footprint" "lib:Diode"
 			(at 101.346 127.762 0)
 			(effects
@@
 			)
 		)
-		(property "Footprint" "kometa:ChocV2"
+		(property "Footprint" "lib:ChocV2"
 			(at 46.736 130.81 0)
 			(effects
@@
 			)
 		)
-		(property "Footprint" "kometa:ChocV2"
+		(property "Footprint" "lib:ChocV2"
 			(at 135.636 111.76 0)
 			(effects
@@
 			)
 		)
-		(property "Footprint" "kometa:Diode"
+		(property "Footprint" "lib:Diode"
 			(at 83.566 108.712 0)
 			(effects
@@
 			)
 		)
-		(property "Footprint" "kometa:ChocV2"
+		(property "Footprint" "lib:ChocV2"
 			(at 117.856 130.81 0)
 			(effects
@@
 			)
 		)
-		(property "Footprint" "kometa:Diode"
+		(property "Footprint" "lib:Diode"
 			(at 119.126 108.712 0)
 			(effects
@@
 			)
 		)
-		(property "Footprint" "kometa:Diode"
+		(property "Footprint" "lib:Diode"
 			(at 136.906 90.932 0)
 			(effects
@@
 			)
 		)
-		(property "Footprint" "kometa:Diode"
+		(property "Footprint" "lib:Diode"
 			(at 101.346 90.932 0)
 			(effects
@@
 			)
 		)
-		(property "Footprint" "kometa:Diode"
+		(property "Footprint" "lib:Diode"
 			(at 65.786 143.002 0)
 			(effects
@@
 			)
 		)
-		(property "Footprint" "kometa:ChocV2"
+		(property "Footprint" "lib:ChocV2"
 			(at 135.636 93.98 0)
 			(effects
@@
 			)
 		)
-		(property "Footprint" "kometa:Diode"
+		(property "Footprint" "lib:Diode"
 			(at 48.006 90.932 0)
 			(effects
@@
 			)
 		)
-		(property "Footprint" "kometa:ChocV2"
+		(property "Footprint" "lib:ChocV2"
 			(at 46.736 146.05 0)
 			(effects
@@
 			)
 		)
-		(property "Footprint" "kometa:Diode"
+		(property "Footprint" "lib:Diode"
 			(at 65.786 90.932 0)
 			(effects
@@
 			)
 		)
-		(property "Footprint" "kometa:Reset"
+		(property "Footprint" "lib:Reset"
 			(at 176.53 119.38 0)
 			(effects
@@
 			)
 		)
-		(property "Footprint" "kometa:Battery"
+		(property "Footprint" "lib:Battery"
 			(at 167.894 89.916 0)
 			(effects
@@
 			)
 		)
-		(property "Footprint" "kometa:Diode"
+		(property "Footprint" "lib:Diode"
 			(at 119.126 90.932 0)
 			(effects
@@
 			)
 		)
-		(property "Footprint" "kometa:Diode"
+		(property "Footprint" "lib:Diode"
 			(at 136.906 127.762 0)
 			(effects
@@
 			)
 		)
-		(property "Footprint" "kometa:ChocV2"
+		(property "Footprint" "lib:ChocV2"
 			(at 117.856 93.98 0)
 			(effects
@@
 			)
 		)
-		(property "Footprint" "kometa:Diode"
+		(property "Footprint" "lib:Diode"
 			(at 48.006 143.002 0)
 			(effects
@@
 			)
 		)
-		(property "Footprint" "kometa:ChocV2"
+		(property "Footprint" "lib:ChocV2"
 			(at 82.296 146.05 0)
 			(effects
@@
 			)
 		)
-		(property "Footprint" "kometa:Diode"
+		(property "Footprint" "lib:Diode"
 			(at 83.566 143.002 0)
 			(effects
@@
 			)
 		)
-		(property "Footprint" "kometa:ChocV2"
+		(property "Footprint" "lib:ChocV2"
 			(at 100.076 111.76 0)
 			(effects
@@
 			)
 		)
-		(property "Footprint" "kometa:ChocV2"
+		(property "Footprint" "lib:ChocV2"
 			(at 100.076 130.81 0)
 			(effects
@@
 			)
 		)
-		(property "Footprint" "kometa:ChocV2"
+		(property "Footprint" "lib:ChocV2"
 			(at 64.516 146.05 0)
 			(effects
@@
 			)
 		)
-		(property "Footprint" "kometa:ChocV2"
+		(property "Footprint" "lib:ChocV2"
 			(at 46.736 93.98 0)
 			(effects
@@
 			)
 		)
-		(property "Footprint" "kometa:Diode"
+		(property "Footprint" "lib:Diode"
 			(at 65.786 108.712 0)
 			(effects
@@
 			)
 		)
-		(property "Footprint" "kometa:ChocV2"
+		(property "Footprint" "lib:ChocV2"
 			(at 82.296 111.76 0)
 			(effects
@@
 			)
 		)
-		(property "Footprint" "kometa:ChocV2"
+		(property "Footprint" "lib:ChocV2"
 			(at 46.736 111.76 0)
 			(effects
@@
 			)
 		)
-		(property "Footprint" "kometa:Diode"
+		(property "Footprint" "lib:Diode"
 			(at 48.006 108.712 0)
 			(effects
@@
 			)
 		)
-		(property "Footprint" "kometa:ChocV2"
+		(property "Footprint" "lib:ChocV2"
 			(at 117.856 111.76 0)
 			(effects
@@
 			)
 		)
-		(property "Footprint" "kometa:Diode"
+		(property "Footprint" "lib:Diode"
 			(at 48.006 127.762 0)
 			(effects
@@
 			)
 		)
-		(property "Footprint" "kometa:ChocV2"
+		(property "Footprint" "lib:ChocV2"
 			(at 64.516 130.81 0)
 			(effects
@@
 			)
 		)
-		(property "Footprint" "kometa:Diode"
+		(property "Footprint" "lib:Diode"
 			(at 119.126 127.762 0)
 			(effects
@@
 			)
 		)
-		(property "Footprint" "kometa:SuperMini"
+		(property "Footprint" "lib:SuperMini"
 			(at 233.68 119.888 0)
 			(effects
@@
 			)
 		)
-		(property "Footprint" "kometa:ChocV2"
+		(property "Footprint" "lib:ChocV2"
 			(at 82.296 93.98 0)
 			(effects
@@
 			)
 		)
-		(property "Footprint" "kometa:ChocV2"
+		(property "Footprint" "lib:ChocV2"
 			(at 82.296 130.81 0)
 			(effects
@@
 			)
 		)
-		(property "Footprint" "kometa:MSK-12C02"
+		(property "Footprint" "lib:MSK-12C02"
 			(at 178.054 91.694 0)
 			(effects
@@
 			)
 		)
-		(property "Footprint" "kometa:Diode"
+		(property "Footprint" "lib:Diode"
 			(at 101.346 108.712 0)
 			(effects
@@
 			)
 		)
-		(property "Footprint" "kometa:Diode"
+		(property "Footprint" "lib:Diode"
 			(at 83.566 90.932 0)
 			(effects
@@
 			)
 		)
-		(property "Footprint" "kometa:ChocV2"
+		(property "Footprint" "lib:ChocV2"
 			(at 100.076 93.98 0)
 			(effects
@@
 			)
 		)
-		(property "Footprint" "kometa:Diode"
+		(property "Footprint" "lib:Diode"
 			(at 65.786 127.762 0)
 			(effects

Commit message: add support choc v1
Parts:
- D22, D23, D24, D25, D26, D27, D28, D29, D30, D31, D32, D33, D34, D35, D36, D37, D38, D39, D40, D41, D42: footprint lib:Diode -> kometa:Diode
- PS_R1: footprint lib:MSK-12C02 -> kometa:MSK-12C02
- PW_R1: footprint lib:Battery -> kometa:Battery
- R_R1: footprint lib:Reset -> kometa:Reset
- SM_R1: footprint lib:SuperMini -> kometa:SuperMini
- SW22, SW23, SW24, SW25, SW26, SW27, SW28, SW29, SW30, SW31, SW32, SW33, SW34, SW35, SW36, SW37, SW38, SW39, SW40, SW41, SW42: footprint lib:ChocV2 -> kometa:ChocV2
Changed lines of the file:
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@@
 			)
 		)
-		(property "Footprint" "lib:ChocV2"
+		(property "Footprint" "kometa:ChocV2"
 			(at 64.516 93.98 0)
 			(effects
@@
 			)
 		)
-		(property "Footprint" "lib:ChocV2"
+		(property "Footprint" "kometa:ChocV2"
 			(at 135.636 130.81 0)
 			(effects
@@
 			)
 		)
-		(property "Footprint" "lib:Diode"
+		(property "Footprint" "kometa:Diode"
 			(at 136.906 108.712 0)
 			(effects
@@
 			)
 		)
-		(property "Footprint" "lib:Diode"
+		(property "Footprint" "kometa:Diode"
 			(at 83.566 127.762 0)
 			(effects
@@
 			)
 		)
-		(property "Footprint" "lib:ChocV2"
+		(property "Footprint" "kometa:ChocV2"
 			(at 64.516 111.76 0)
 			(effects
@@
 			)
 		)
-		(property "Footprint" "lib:Diode"
+		(property "Footprint" "kometa:Diode"
 			(at 101.346 127.762 0)
 			(effects
@@
 			)
 		)
-		(property "Footprint" "lib:ChocV2"
+		(property "Footprint" "kometa:ChocV2"
 			(at 46.736 130.81 0)
 			(effects
@@
 			)
 		)
-		(property "Footprint" "lib:ChocV2"
+		(property "Footprint" "kometa:ChocV2"
 			(at 135.636 111.76 0)
 			(effects
@@
 			)
 		)
-		(property "Footprint" "lib:Diode"
+		(property "Footprint" "kometa:Diode"
 			(at 83.566 108.712 0)
 			(effects
@@
 			)
 		)
-		(property "Footprint" "lib:ChocV2"
+		(property "Footprint" "kometa:ChocV2"
 			(at 117.856 130.81 0)
 			(effects
@@
 			)
 		)
-		(property "Footprint" "lib:Diode"
+		(property "Footprint" "kometa:Diode"
 			(at 119.126 108.712 0)
 			(effects
@@
 			)
 		)
-		(property "Footprint" "lib:Diode"
+		(property "Footprint" "kometa:Diode"
 			(at 136.906 90.932 0)
 			(effects
@@
 			)
 		)
-		(property "Footprint" "lib:Diode"
+		(property "Footprint" "kometa:Diode"
 			(at 101.346 90.932 0)
 			(effects
@@
 			)
 		)
-		(property "Footprint" "lib:Diode"
+		(property "Footprint" "kometa:Diode"
 			(at 65.786 143.002 0)
 			(effects
@@
 			)
 		)
-		(property "Footprint" "lib:ChocV2"
+		(property "Footprint" "kometa:ChocV2"
 			(at 135.636 93.98 0)
 			(effects
@@
 			)
 		)
-		(property "Footprint" "lib:Diode"
+		(property "Footprint" "kometa:Diode"
 			(at 48.006 90.932 0)
 			(effects
@@
 			)
 		)
-		(property "Footprint" "lib:ChocV2"
+		(property "Footprint" "kometa:ChocV2"
 			(at 46.736 146.05 0)
 			(effects
@@
 			)
 		)
-		(property "Footprint" "lib:Diode"
+		(property "Footprint" "kometa:Diode"
 			(at 65.786 90.932 0)
 			(effects
@@
 			)
 		)
-		(property "Footprint" "lib:Reset"
+		(property "Footprint" "kometa:Reset"
 			(at 176.53 119.38 0)
 			(effects
@@
 			)
 		)
-		(property "Footprint" "lib:Battery"
+		(property "Footprint" "kometa:Battery"
 			(at 167.894 89.916 0)
 			(effects
@@
 			)
 		)
-		(property "Footprint" "lib:Diode"
+		(property "Footprint" "kometa:Diode"
 			(at 119.126 90.932 0)
 			(effects
@@
 			)
 		)
-		(property "Footprint" "lib:Diode"
+		(property "Footprint" "kometa:Diode"
 			(at 136.906 127.762 0)
 			(effects
@@
 			)
 		)
-		(property "Footprint" "lib:ChocV2"
+		(property "Footprint" "kometa:ChocV2"
 			(at 117.856 93.98 0)
 			(effects
@@
 			)
 		)
-		(property "Footprint" "lib:Diode"
+		(property "Footprint" "kometa:Diode"
 			(at 48.006 143.002 0)
 			(effects
@@
 			)
 		)
-		(property "Footprint" "lib:ChocV2"
+		(property "Footprint" "kometa:ChocV2"
 			(at 82.296 146.05 0)
 			(effects
@@
 			)
 		)
-		(property "Footprint" "lib:Diode"
+		(property "Footprint" "kometa:Diode"
 			(at 83.566 143.002 0)
 			(effects
@@
 			)
 		)
-		(property "Footprint" "lib:ChocV2"
+		(property "Footprint" "kometa:ChocV2"
 			(at 100.076 111.76 0)
 			(effects
@@
 			)
 		)
-		(property "Footprint" "lib:ChocV2"
+		(property "Footprint" "kometa:ChocV2"
 			(at 100.076 130.81 0)
 			(effects
@@
 			)
 		)
-		(property "Footprint" "lib:ChocV2"
+		(property "Footprint" "kometa:ChocV2"
 			(at 64.516 146.05 0)
 			(effects
@@
 			)
 		)
-		(property "Footprint" "lib:ChocV2"
+		(property "Footprint" "kometa:ChocV2"
 			(at 46.736 93.98 0)
 			(effects
@@
 			)
 		)
-		(property "Footprint" "lib:Diode"
+		(property "Footprint" "kometa:Diode"
 			(at 65.786 108.712 0)
 			(effects
@@
 			)
 		)
-		(property "Footprint" "lib:ChocV2"
+		(property "Footprint" "kometa:ChocV2"
 			(at 82.296 111.76 0)
 			(effects
@@
 			)
 		)
-		(property "Footprint" "lib:ChocV2"
+		(property "Footprint" "kometa:ChocV2"
 			(at 46.736 111.76 0)
 			(effects
@@
 			)
 		)
-		(property "Footprint" "lib:Diode"
+		(property "Footprint" "kometa:Diode"
 			(at 48.006 108.712 0)
 			(effects
@@
 			)
 		)
-		(property "Footprint" "lib:ChocV2"
+		(property "Footprint" "kometa:ChocV2"
 			(at 117.856 111.76 0)
 			(effects
@@
 			)
 		)
-		(property "Footprint" "lib:Diode"
+		(property "Footprint" "kometa:Diode"
 			(at 48.006 127.762 0)
 			(effects
@@
 			)
 		)
-		(property "Footprint" "lib:ChocV2"
+		(property "Footprint" "kometa:ChocV2"
 			(at 64.516 130.81 0)
 			(effects
@@
 			)
 		)
-		(property "Footprint" "lib:Diode"
+		(property "Footprint" "kometa:Diode"
 			(at 119.126 127.762 0)
 			(effects
@@
 			)
 		)
-		(property "Footprint" "lib:SuperMini"
+		(property "Footprint" "kometa:SuperMini"
 			(at 233.68 119.888 0)
 			(effects
@@
 			)
 		)
-		(property "Footprint" "lib:ChocV2"
+		(property "Footprint" "kometa:ChocV2"
 			(at 82.296 93.98 0)
 			(effects
@@
 			)
 		)
-		(property "Footprint" "lib:ChocV2"
+		(property "Footprint" "kometa:ChocV2"
 			(at 82.296 130.81 0)
 			(effects
@@
 			)
 		)
-		(property "Footprint" "lib:MSK-12C02"
+		(property "Footprint" "kometa:MSK-12C02"
 			(at 178.054 91.694 0)
 			(effects
@@
 			)
 		)
-		(property "Footprint" "lib:Diode"
+		(property "Footprint" "kometa:Diode"
 			(at 101.346 108.712 0)
 			(effects
@@
 			)
 		)
-		(property "Footprint" "lib:Diode"
+		(property "Footprint" "kometa:Diode"
 			(at 83.566 90.932 0)
 			(effects
@@
 			)
 		)
-		(property "Footprint" "lib:ChocV2"
+		(property "Footprint" "kometa:ChocV2"
 			(at 100.076 93.98 0)
 			(effects
@@
 			)
 		)
-		(property "Footprint" "lib:Diode"
+		(property "Footprint" "kometa:Diode"
 			(at 65.786 127.762 0)
 			(effects
