File: PCB/left.kicad_sch (KiCad schematic)
At the start: 47 parts

Commit message: Remove ks27/ks33 support, fix mcu board cutout
Parts:
- SW1, SW10, SW11, SW12, SW13, SW14, SW15, SW16, SW17, SW18, SW19, SW2, SW20, SW21, SW3, SW4, SW5, SW6, SW7, SW8, SW9: footprint kometa:SW_Hotswap_Kailh_Choc_V1V2_with_KS27_KS33 -> kometa:SW_Hotswap_Kailh_Choc_V1V2
Changed lines of the file:
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@@
 			)
 		)
-		(property "Footprint" "kometa:SW_Hotswap_Kailh_Choc_V1V2_with_KS27_KS33"
+		(property "Footprint" "kometa:SW_Hotswap_Kailh_Choc_V1V2"
 			(at 79.756 105.41 0)
 			(effects
@@
 			)
 		)
-		(property "Footprint" "kometa:SW_Hotswap_Kailh_Choc_V1V2_with_KS27_KS33"
+		(property "Footprint" "kometa:SW_Hotswap_Kailh_Choc_V1V2"
 			(at 136.906 105.41 0)
 			(effects
@@
 			)
 		)
-		(property "Footprint" "kometa:SW_Hotswap_Kailh_Choc_V1V2_with_KS27_KS33"
+		(property "Footprint" "kometa:SW_Hotswap_Kailh_Choc_V1V2"
 			(at 41.656 86.36 0)
 			(effects
@@
 			)
 		)
-		(property "Footprint" "kometa:SW_Hotswap_Kailh_Choc_V1V2_with_KS27_KS33"
+		(property "Footprint" "kometa:SW_Hotswap_Kailh_Choc_V1V2"
 			(at 136.906 86.36 0)
 			(effects
@@
 			)
 		)
-		(property "Footprint" "kometa:SW_Hotswap_Kailh_Choc_V1V2_with_KS27_KS33"
+		(property "Footprint" "kometa:SW_Hotswap_Kailh_Choc_V1V2"
 			(at 98.806 124.46 0)
 			(effects
@@
 			)
 		)
-		(property "Footprint" "kometa:SW_Hotswap_Kailh_Choc_V1V2_with_KS27_KS33"
+		(property "Footprint" "kometa:SW_Hotswap_Kailh_Choc_V1V2"
 			(at 136.906 124.46 0)
 			(effects
@@
 			)
 		)
-		(property "Footprint" "kometa:SW_Hotswap_Kailh_Choc_V1V2_with_KS27_KS33"
+		(property "Footprint" "kometa:SW_Hotswap_Kailh_Choc_V1V2"
 			(at 60.706 86.36 0)
 			(effects
@@
 			)
 		)
-		(property "Footprint" "kometa:SW_Hotswap_Kailh_Choc_V1V2_with_KS27_KS33"
+		(property "Footprint" "kometa:SW_Hotswap_Kailh_Choc_V1V2"
 			(at 117.856 144.78 0)
 			(effects
@@
 			)
 		)
-		(property "Footprint" "kometa:SW_Hotswap_Kailh_Choc_V1V2_with_KS27_KS33"
+		(property "Footprint" "kometa:SW_Hotswap_Kailh_Choc_V1V2"
 			(at 117.856 105.41 0)
 			(effects
@@
 			)
 		)
-		(property "Footprint" "kometa:SW_Hotswap_Kailh_Choc_V1V2_with_KS27_KS33"
+		(property "Footprint" "kometa:SW_Hotswap_Kailh_Choc_V1V2"
 			(at 79.756 86.36 0)
 			(effects
@@
 			)
 		)
-		(property "Footprint" "kometa:SW_Hotswap_Kailh_Choc_V1V2_with_KS27_KS33"
+		(property "Footprint" "kometa:SW_Hotswap_Kailh_Choc_V1V2"
 			(at 117.856 86.36 0)
 			(effects
@@
 			)
 		)
-		(property "Footprint" "kometa:SW_Hotswap_Kailh_Choc_V1V2_with_KS27_KS33"
+		(property "Footprint" "kometa:SW_Hotswap_Kailh_Choc_V1V2"
 			(at 41.656 124.46 0)
 			(effects
@@
 			)
 		)
-		(property "Footprint" "kometa:SW_Hotswap_Kailh_Choc_V1V2_with_KS27_KS33"
+		(property "Footprint" "kometa:SW_Hotswap_Kailh_Choc_V1V2"
 			(at 60.706 124.46 0)
 			(effects
@@
 			)
 		)
-		(property "Footprint" "kometa:SW_Hotswap_Kailh_Choc_V1V2_with_KS27_KS33"
+		(property "Footprint" "kometa:SW_Hotswap_Kailh_Choc_V1V2"
 			(at 98.806 86.36 0)
 			(effects
@@
 			)
 		)
-		(property "Footprint" "kometa:SW_Hotswap_Kailh_Choc_V1V2_with_KS27_KS33"
+		(property "Footprint" "kometa:SW_Hotswap_Kailh_Choc_V1V2"
 			(at 117.856 124.46 0)
 			(effects
@@
 			)
 		)
-		(property "Footprint" "kometa:SW_Hotswap_Kailh_Choc_V1V2_with_KS27_KS33"
+		(property "Footprint" "kometa:SW_Hotswap_Kailh_Choc_V1V2"
 			(at 98.806 144.78 0)
 			(effects
@@
 			)
 		)
-		(property "Footprint" "kometa:SW_Hotswap_Kailh_Choc_V1V2_with_KS27_KS33"
+		(property "Footprint" "kometa:SW_Hotswap_Kailh_Choc_V1V2"
 			(at 41.656 105.41 0)
 			(effects
@@
 			)
 		)
-		(property "Footprint" "kometa:SW_Hotswap_Kailh_Choc_V1V2_with_KS27_KS33"
+		(property "Footprint" "kometa:SW_Hotswap_Kailh_Choc_V1V2"
 			(at 60.706 105.41 0)
 			(effects
@@
 			)
 		)
-		(property "Footprint" "kometa:SW_Hotswap_Kailh_Choc_V1V2_with_KS27_KS33"
+		(property "Footprint" "kometa:SW_Hotswap_Kailh_Choc_V1V2"
 			(at 98.806 105.41 0)
 			(effects
@@
 			)
 		)
-		(property "Footprint" "kometa:SW_Hotswap_Kailh_Choc_V1V2_with_KS27_KS33"
+		(property "Footprint" "kometa:SW_Hotswap_Kailh_Choc_V1V2"
 			(at 79.756 124.46 0)
 			(effects
@@
 			)
 		)
-		(property "Footprint" "kometa:SW_Hotswap_Kailh_Choc_V1V2_with_KS27_KS33"
+		(property "Footprint" "kometa:SW_Hotswap_Kailh_Choc_V1V2"
 			(at 136.906 144.78 0)
 			(effects
