File: PCB/right.kicad_sch (KiCad schematic)
At the start: 47 parts

Commit message: Remove ks27/ks33 support, fix mcu board cutout
Parts:
- SW22, SW23, SW24, SW25, SW26, SW27, SW28, SW29, SW30, SW31, SW32, SW33, SW34, SW35, SW36, SW37, SW38, SW39, SW40, SW41, SW42: footprint kometa:SW_Hotswap_Kailh_Choc_V1V2_with_KS27_KS33 -> kometa:SW_Hotswap_Kailh_Choc_V1V2
Changed lines of the file:
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@@
 			)
 		)
-		(property "Footprint" "kometa:SW_Hotswap_Kailh_Choc_V1V2_with_KS27_KS33"
+		(property "Footprint" "kometa:SW_Hotswap_Kailh_Choc_V1V2"
 			(at 64.516 93.98 0)
 			(effects
@@
 			)
 		)
-		(property "Footprint" "kometa:SW_Hotswap_Kailh_Choc_V1V2_with_KS27_KS33"
+		(property "Footprint" "kometa:SW_Hotswap_Kailh_Choc_V1V2"
 			(at 135.636 130.81 0)
 			(effects
@@
 			)
 		)
-		(property "Footprint" "kometa:SW_Hotswap_Kailh_Choc_V1V2_with_KS27_KS33"
+		(property "Footprint" "kometa:SW_Hotswap_Kailh_Choc_V1V2"
 			(at 64.516 111.76 0)
 			(effects
@@
 			)
 		)
-		(property "Footprint" "kometa:SW_Hotswap_Kailh_Choc_V1V2_with_KS27_KS33"
+		(property "Footprint" "kometa:SW_Hotswap_Kailh_Choc_V1V2"
 			(at 46.736 130.81 0)
 			(effects
@@
 			)
 		)
-		(property "Footprint" "kometa:SW_Hotswap_Kailh_Choc_V1V2_with_KS27_KS33"
+		(property "Footprint" "kometa:SW_Hotswap_Kailh_Choc_V1V2"
 			(at 135.636 111.76 0)
 			(effects
@@
 			)
 		)
-		(property "Footprint" "kometa:SW_Hotswap_Kailh_Choc_V1V2_with_KS27_KS33"
+		(property "Footprint" "kometa:SW_Hotswap_Kailh_Choc_V1V2"
 			(at 117.856 130.81 0)
 			(effects
@@
 			)
 		)
-		(property "Footprint" "kometa:SW_Hotswap_Kailh_Choc_V1V2_with_KS27_KS33"
+		(property "Footprint" "kometa:SW_Hotswap_Kailh_Choc_V1V2"
 			(at 135.636 93.98 0)
 			(effects
@@
 			)
 		)
-		(property "Footprint" "kometa:SW_Hotswap_Kailh_Choc_V1V2_with_KS27_KS33"
+		(property "Footprint" "kometa:SW_Hotswap_Kailh_Choc_V1V2"
 			(at 46.736 146.05 0)
 			(effects
@@
 			)
 		)
-		(property "Footprint" "kometa:SW_Hotswap_Kailh_Choc_V1V2_with_KS27_KS33"
+		(property "Footprint" "kometa:SW_Hotswap_Kailh_Choc_V1V2"
 			(at 117.856 93.98 0)
 			(effects
@@
 			)
 		)
-		(property "Footprint" "kometa:SW_Hotswap_Kailh_Choc_V1V2_with_KS27_KS33"
+		(property "Footprint" "kometa:SW_Hotswap_Kailh_Choc_V1V2"
 			(at 82.296 146.05 0)
 			(effects
@@
 			)
 		)
-		(property "Footprint" "kometa:SW_Hotswap_Kailh_Choc_V1V2_with_KS27_KS33"
+		(property "Footprint" "kometa:SW_Hotswap_Kailh_Choc_V1V2"
 			(at 100.076 111.76 0)
 			(effects
@@
 			)
 		)
-		(property "Footprint" "kometa:SW_Hotswap_Kailh_Choc_V1V2_with_KS27_KS33"
+		(property "Footprint" "kometa:SW_Hotswap_Kailh_Choc_V1V2"
 			(at 100.076 130.81 0)
 			(effects
@@
 			)
 		)
-		(property "Footprint" "kometa:SW_Hotswap_Kailh_Choc_V1V2_with_KS27_KS33"
+		(property "Footprint" "kometa:SW_Hotswap_Kailh_Choc_V1V2"
 			(at 64.516 146.05 0)
 			(effects
@@
 			)
 		)
-		(property "Footprint" "kometa:SW_Hotswap_Kailh_Choc_V1V2_with_KS27_KS33"
+		(property "Footprint" "kometa:SW_Hotswap_Kailh_Choc_V1V2"
 			(at 46.736 93.98 0)
 			(effects
@@
 			)
 		)
-		(property "Footprint" "kometa:SW_Hotswap_Kailh_Choc_V1V2_with_KS27_KS33"
+		(property "Footprint" "kometa:SW_Hotswap_Kailh_Choc_V1V2"
 			(at 82.296 111.76 0)
 			(effects
@@
 			)
 		)
-		(property "Footprint" "kometa:SW_Hotswap_Kailh_Choc_V1V2_with_KS27_KS33"
+		(property "Footprint" "kometa:SW_Hotswap_Kailh_Choc_V1V2"
 			(at 46.736 111.76 0)
 			(effects
@@
 			)
 		)
-		(property "Footprint" "kometa:SW_Hotswap_Kailh_Choc_V1V2_with_KS27_KS33"
+		(property "Footprint" "kometa:SW_Hotswap_Kailh_Choc_V1V2"
 			(at 117.856 111.76 0)
 			(effects
@@
 			)
 		)
-		(property "Footprint" "kometa:SW_Hotswap_Kailh_Choc_V1V2_with_KS27_KS33"
+		(property "Footprint" "kometa:SW_Hotswap_Kailh_Choc_V1V2"
 			(at 64.516 130.81 0)
 			(effects
@@
 			)
 		)
-		(property "Footprint" "kometa:SW_Hotswap_Kailh_Choc_V1V2_with_KS27_KS33"
+		(property "Footprint" "kometa:SW_Hotswap_Kailh_Choc_V1V2"
 			(at 82.296 93.98 0)
 			(effects
@@
 			)
 		)
-		(property "Footprint" "kometa:SW_Hotswap_Kailh_Choc_V1V2_with_KS27_KS33"
+		(property "Footprint" "kometa:SW_Hotswap_Kailh_Choc_V1V2"
 			(at 82.296 130.81 0)
 			(effects
@@
 			)
 		)
-		(property "Footprint" "kometa:SW_Hotswap_Kailh_Choc_V1V2_with_KS27_KS33"
+		(property "Footprint" "kometa:SW_Hotswap_Kailh_Choc_V1V2"
 			(at 100.076 93.98 0)
 			(effects
